File: esp32.sch (KiCad schematic (older format))
At the start: 34 parts, among them J1 Conn_01x02_Male, J2 DM3AT-SF-PEJM5(40), Q1 DMG2305UX-7, U1 ESP32-WROOM-32, Y1 LFXTAL009709Bulk

Commit message: changed to a more basic variant of the esp32
Parts:
- removed C1, C2, C4: 100n/25V, bytewerk_capacitors:C_0603_1608Metric, symbol bytewerk-discrete:C
- removed C3, C5: 10u/25V, bytewerk_capacitors:C_0805_2012Metric, symbol bytewerk-discrete:C
- removed C6, C7: C, bytewerk_capacitors:C_0603_1608Metric, symbol bytewerk-discrete:C
- removed D3: BAT54C, Package_TO_SOT_SMD:SOT-23, symbol Diode:BAT54C
- removed J2: DM3AT-SF-PEJM5(40), Connector_Card:microSD_HC_Hirose_DM3AT-SF-PEJM5, symbol Connector:Micro_SD_Card_Det
- removed L1, L2: L, Inductor_SMD:L_0603_1608Metric, symbol Device:L
- removed Q1: DMG2305UX-7, Package_TO_SOT_SMD:SOT-23, symbol Device:Q_PMOS_GSD
- removed R10: 10R, bytewerk_resistors:R_0603_1608Metric, symbol bytewerk-discrete:R
- removed R11, R12, R13, R9: 33R, bytewerk_resistors:R_0603_1608Metric, symbol bytewerk-discrete:R
- removed R14: 200R, bytewerk_resistors:R_0603_1608Metric, symbol bytewerk-discrete:R
- removed R15, R3, R4, R5, R6, R7, R8: 10k, bytewerk_resistors:R_0603_1608Metric, symbol bytewerk-discrete:R
- removed U1: ESP32-WROOM-32, bytewerk-esp32:ESP32-WROOM-32, symbol bytewerk-esp32:ESP32-WROOM-32
- removed Y1: LFXTAL009709Bulk, Crystal:Crystal_SMD_3215-2Pin_3.2x1.5mm, symbol Device:Crystal
- added U1: ESP32-DevKitC-32D, bytewerk-esp32:ESP32-DevKitC-32D, symbol bytewerk-esp32:ESP32-DevKitC-32D
- J1: footprint Connector_PinHeader_2.54mm:PinHeader_1x02_P2.54mm_Horizontal -> Connector_PinHeader_2.54mm:PinHeader_1x02_P2.54mm_Vertical
Connections:
- net labels added: RXD, TXD
- net labels removed: BOOT, DET_A, DET_B, ESP_EN, IO0, SD_CLK, SD_CMD, SD_DAT0, SD_DAT1, SD_DAT2, SD_DAT3, SD_EN, SD_VDD, UART_USB_RX, UART_USB_TX
- wire segments 133 -> 30
- no-connect marks 9 -> 25
Other:
- note added: "Remove diode D3 from ESP32-DevKitC\nhttps://dl.espressif.com/dl/schematics/esp32_devkitc_v4-sch-20180607a.pdf"
- note removed: "0: SPI Boot\n1: Download Boot"
- note removed: "activate internal pullup in \nuser programm on GPIO12"
- note removed: "using two pins for lower quiescent current"
