File: power_supply.sch (KiCad schematic (older format))
At the start: 22 parts, among them J3 DB9_Male, U4 LT8607

Commit message: changed to a more basic variant of the esp32
Parts:
- removed C10, C15, C16: 10u/25V, bytewerk_capacitors:C_0805_2012Metric, symbol bytewerk-discrete:C
- removed C11: 1u/25V, bytewerk_capacitors:C_0603_1608Metric, symbol bytewerk-discrete:C
- removed C12: 10n/25V, bytewerk_capacitors:C_0603_1608Metric, symbol bytewerk-discrete:C
- removed C13: 100n/25V, bytewerk_capacitors:C_0603_1608Metric, symbol bytewerk-discrete:C
- removed C14: 10p/50V, bytewerk_capacitors:C_0603_1608Metric, symbol bytewerk-discrete:C
- removed L3: XFL3012-222ME, bytewerk-inductors:L_Coilcraft_XLF3012, symbol Device:L
- removed R24, R32: 1M, bytewerk_resistors:R_0603_1608Metric, symbol bytewerk-discrete:R
- removed R25: 120k, bytewerk_resistors:R_0603_1608Metric, symbol bytewerk-discrete:R
- removed R28: n.b., bytewerk_resistors:R_0603_1608Metric, symbol bytewerk-discrete:R
- removed R29: 18k, bytewerk_resistors:R_0603_1608Metric, symbol bytewerk-discrete:R
- removed R30: 200R, bytewerk_resistors:R_0603_1608Metric, symbol bytewerk-discrete:R
- removed R31: 82k, bytewerk_resistors:R_0603_1608Metric, symbol bytewerk-discrete:R
- removed R33: 309k, bytewerk_resistors:R_0603_1608Metric, symbol bytewerk-discrete:R
- removed U4: LT8607, Package_SO:MSOP-10-1EP_3x3mm_P0.5mm_EP1.68x1.88mm, symbol bytewerk-vreg:LT8607
- added U4: OKI-78SR, bytewerk-TO-packages:TO-220-3_Horizontal_TabDown, symbol bytewerk-vreg:OKI-78SR
- D4: MPN (none) -> NUP2105L
Connections:
- net labels removed: Power_Good
- wire segments 80 -> 25
Other:
- note added: "add heat shrink tube to OKI"
- note removed: "Voltage regulator will be \nshut down below 9V of V_BAT\nVin(en) around 9,33V"
