File: usb_uart.sch (KiCad schematic (older format))
At the start: 20 parts, among them J4 USB_B_Micro, Q2 BC817, Q3 BC817, U5 USBLC6-2SC6, U6 CP2102N-A01-GQFN24

Commit message: changed to a more basic variant of the esp32
Parts:
- J4: MPN (none) -> 629105150521
- Q2, Q3: MPN (none) -> BC817-40WT1G
- U5: MPN (none) -> USBLC6-2SC6
- U6: MPN (none) -> CP2102N-A01-GQFN24
Changed lines of the file:
@@
 encoding utf-8
 Sheet 5 5
-Title "WIFI-CAN-Dongle"
-Date "2018-09-30"
+Title "WIFI-CAN-Dongle Basic"
+Date "2018-10-03"
 Rev "v1.0"
-Comp ""
+Comp "bytewerk - www.bytewerk.org"
 Comment1 ""
 Comment2 "Stephan Hültl"
@@
 F 2 "Connector_USB:USB_Micro-B_Wuerth_629105150521_CircularHoles" H 1300 2700 50  0001 C CNN
 F 3 "~" H 1300 2700 50  0001 C CNN
+F 4 "629105150521" H 1150 2750 50  0001 C CNN "MPN"
 	1    1150 2750
 	1    0    0    -1
@@
 F 2 "Package_TO_SOT_SMD:SOT-23-6" H 1000 5200 50  0001 C CNN
 F 3 "http://www2.st.com/resource/en/datasheet/CD00050750.pdf" H 1950 5150 50  0001 C CNN
+F 4 "USBLC6-2SC6" H 1750 4800 50  0001 C CNN "MPN"
 	1    1750 4800
 	1    0    0    -1
@@
 F 2 "Package_DFN_QFN:QFN-24-1EP_4x4mm_P0.5mm_EP2.6x2.6mm" H 6750 2500 50  0001 L CNN
 F 3 "http://www.silabs.com/support%20documents/technicaldocs/cp2102n-datasheet.pdf" H 6350 2250 50  0001 C CNN
+F 4 "CP2102N-A01-GQFN24" H 6300 3300 50  0001 C CNN "MPN"
 	1    6300 3300
 	1    0    0    -1
@@
 F 2 "Package_TO_SOT_SMD:SOT-23" H 9350 4475 50  0001 L CIN
 F 3 "http://www.fairchildsemi.com/ds/BC/BC817.pdf" H 9150 4550 50  0001 L CNN
+F 4 "BC817-40WT1G" H 9150 4550 50  0001 C CNN "MPN"
 	1    9150 4550
 	1    0    0    -1
@@
 F 2 "Package_TO_SOT_SMD:SOT-23" H 9350 5375 50  0001 L CIN
 F 3 "http://www.fairchildsemi.com/ds/BC/BC817.pdf" H 9150 5450 50  0001 L CNN
+F 4 "BC817-40WT1G" H 9150 5450 50  0001 C CNN "MPN"
 	1    9150 5450
 	1    0    0    1
